Commit message: Update firmware, fix physical params, and tune Nav2 stack
- Replace firmware with teammate's version (correct CAN API IDs, duty cycle
  mode, PID tuning commands, encoder keepalive, bus voltage monitoring)
- Fix wheel_separation 0.508→0.730m and robot_radius 0.35→0.46m from
  actual robot measurements (32.5" square base, 28.75" track-to-track)
- Fix right_motor_inverted to false (direction set in SparkMAX app)
- Fix acceleration limit mismatch: MPPI, velocity_smoother, and
  diff_drive_controller now all use 1.0 m/s² linear, 3.0 rad/s² angular
- Fix odom_topic in bt_navigator and velocity_smoother to use
  /diff_drive_controller/odom instead of /odom
- Switch velocity_smoother to CLOSED_LOOP for real odometry feedback
- Reduce MPPI PathAlignCritic weight 14→10 and wz_std 0.4→0.2 to
  prevent diff drive wobbling
- Set PreferForwardCritic always active (threshold 0.5→0.0)
- Match angular velocity limit to 1.9 rad/s across all packages
- Forward serial_port arg through teleop.launch.py to igvc_control
- Sync sim nav2 params with real nav2 params

Co-Authored-By: Claude Opus 4.6 <noreply@anthropic.com>

File: src/igvc_control/config/igvc.urdf.xacro (robot description, xacro)
@@ -4,10 +4,10 @@
   <xacro:arg name="serial_port" default="/dev/ttyACM0" />
   <!-- Drivetrain parameters -->
-  <xacro:property name="wheel_separation" value="0.508" />
+  <xacro:property name="wheel_separation" value="0.730" />
   <xacro:property name="wheel_radius"     value="0.0345" />
   <!-- Base link -->
   <link name="base_link">
     <visual>
-      <geometry><box size="0.6 0.5 0.2" /></geometry>
+      <geometry><box size="0.826 0.826 0.2" /></geometry>
     </visual>
   </link>
@@ -52,5 +52,5 @@
       <param name="max_motor_rpm">3000</param>
       <param name="left_motor_inverted">false</param>
-      <param name="right_motor_inverted">true</param>
+      <param name="right_motor_inverted">false</param>
     </hardware>
     <joint name="left_wheel_joint">

File: src/igvc_simulation/config/igvc_sim.urdf.xacro (robot description, xacro)
@@ -2,10 +2,10 @@
 <robot xmlns:xacro="http://www.ros.org/wiki/xacro" name="igvc_sim">
   <!-- Drivetrain parameters — must match igvc_control values -->
-  <xacro:property name="wheel_separation" value="0.508" />
+  <xacro:property name="wheel_separation" value="0.730" />
   <xacro:property name="wheel_radius"     value="0.0345" />
   <!-- Base link -->
   <link name="base_link">
     <visual>
-      <geometry><box size="0.6 0.5 0.2" /></geometry>
+      <geometry><box size="0.826 0.826 0.2" /></geometry>
       <material name="grey"><color rgba="0.5 0.5 0.5 1" /></material>
     </visual>
